Commit message: Add tf results

File: turtlebot3_description/urdf/turtlebot3_burger.urdf (robot description, URDF)
Before this commit: robot turtlebot3_burger, 9 links, 8 joints
Links:
- removed link velodyne
- removed link velodyne_base_link
Joints:
- removed joint velodyne_base_mount_joint
- removed joint velodyne_base_scan_joint
